File: 40board k6/40board k6.kicad_sch (KiCad schematic)
At the start: 0 parts

Commit message: Added Marbastlib and annotations
Parts:
- added C1, C2, C3: 0.1uF, Capacitor_SMD:C_0805_2012Metric, symbol Device:C_Small
- added C4, C5: 22pF, Capacitor_SMD:C_0805_2012Metric, symbol Device:C_Small
- added C6: 10uF, Capacitor_SMD:C_0805_2012Metric, symbol Device:C_Small
- added C7: 1uF, Diode_SMD:D_0805_2012Metric, symbol Device:C_Small
- added D1, D10, D11, D12, D13, D14, D15, D16, D17, D18, D19, D2, D20, D21, D22, D23, D24, D25, D26, D27, D28, D29, D3, D30, D31, D32, D33, D34, D35, D36, D37, D38, D39, D4, D40, D41, D42, D43, D44, D45, D46, D5, D6, D7, D8, D9: D_Small, Diode_SMD:D_SOD-123, symbol Device:D_Small
- added F1: 500mA, Fuse:Fuse_1206_3216Metric, symbol Device:Polyfuse_Small
- added J1: USB_C_Receptacle_USB2.0, marbastlib-various:USB_C_Receptacle_HRO_TYPE-C-31-M-14, symbol Connector:USB_C_Receptacle_USB2.0
- added MX1, MX10, MX11, MX12, MX13, MX14, MX15, MX16, MX17, MX18, MX19, MX2, MX20, MX21, MX22, MX23, MX24, MX25, MX26, MX27, MX28, MX29, MX3, MX30, MX31, MX32, MX33, MX34, MX35, MX36, MX37, MX38, MX39, MX4, MX40, MX41, MX42, MX43, MX44, MX45, MX46, MX5, MX6, MX7, MX8, MX9: MX-NoLED, Kailh_Choc:KailhChoc-1U, symbol MX_Alps_Hybrid:MX-NoLED
- added R1, R2: 22, Resistor_SMD:R_0805_2012Metric, symbol Device:R_Small
- added R3, R4: 10k, Resistor_SMD:R_0805_2012Metric, symbol Device:R_Small
- added R5, R6: 5.1k, Resistor_SMD:R_0805_2012Metric, symbol Device:R_Small
- added SW1: SW_Push, random-keyboard-parts:SKQG-1155865, symbol Switch:SW_Push
- added SW2: RotaryEncoder, Rotary_Encoder:RotaryEncoder_Alps_EC12E_Vertical_H20mm, symbol Device:RotaryEncoder
- added U1: ATmega32U4-M, Package_DFN_QFN:QFN-44-1EP_7x7mm_P0.5mm_EP5.2x5.2mm, symbol MCU_Microchip_ATmega:ATmega32U4-M
- added Y1: 16MHz, Crystal:Crystal_SMD_3225-4Pin_3.2x2.5mm, symbol Device:Crystal_GND24_Small
Connections:
- new net: D37.2 (A), MX37.2 (ROW)
- new net: D12.2 (A), MX12.2 (ROW)
- new net: D2.2 (A), MX2.2 (ROW)
- new net: D3.2 (A), MX3.2 (ROW)
- new net: D41.2 (A), MX41.2 (ROW)
- new net: D19.2 (A), MX19.2 (ROW)
- new net: R2.2, U1.4 (D+)
- new net: D6.2 (A), MX6.2 (ROW)
- new net: D14.2 (A), MX14.2 (ROW)
- new net: D24.2 (A), MX24.2 (ROW)
- new net: D46.2 (A), MX46.2 (ROW)
- new net: D1.2 (A), MX1.2 (ROW)
- new net: D42.2 (A), MX42.2 (ROW)
- new net: D15.2 (A), MX15.2 (ROW)
- new net: D36.2 (A), MX36.2 (ROW)
- new net: D10.2 (A), MX10.2 (ROW)
- new net: D18.2 (A), MX18.2 (ROW)
- new net: D43.2 (A), MX43.2 (ROW)
- new net: D11.2 (A), MX11.2 (ROW)
- new net: D26.2 (A), MX26.2 (ROW)
- new net: D17.2 (A), MX17.2 (ROW)
- new net: D39.2 (A), MX39.2 (ROW)
- new net: D21.2 (A), MX21.2 (ROW)
- new net: D13.2 (A), MX13.2 (ROW)
- new net: D38.2 (A), MX38.2 (ROW)
- new net: C7.1, U1.6 (UCAP)
- new net: D34.2 (A), MX34.2 (ROW)
- new net: D35.2 (A), MX35.2 (ROW)
- new net: D5.2 (A), MX5.2 (ROW)
- new net: D40.2 (A), MX40.2 (ROW)
- new net: D32.2 (A), MX32.2 (ROW)
- new net: D27.2 (A), MX27.2 (ROW)
- new net: D7.2 (A), MX7.2 (ROW)
- new net: J1.A5 (CC1), R6.1
- new net: C4.2, U1.17 (XTAL1), Y1.1
- new net: D9.2 (A), MX9.2 (ROW)
- new net: D30.2 (A), MX30.2 (ROW)
- new net: D8.2 (A), MX8.2 (ROW)
- new net: D16.2 (A), MX16.2 (ROW)
- new net: D4.2 (A), MX4.2 (ROW)
- new net: D33.2 (A), MX33.2 (ROW)
- new net: D20.2 (A), MX20.2 (ROW)
- new net: J1.B5 (CC2), R5.1
- new net: D45.2 (A), MX45.2 (ROW)
- new net: D22.2 (A), MX22.2 (ROW)
- new net: R3.2, SW1.2, U1.13 (~{RESET})
- new net: C5.2, U1.16 (XTAL2), Y1.3
- new net: R1.2, U1.3 (D-)
- new net: R4.1, U1.33 (~{HWB}/PE2)
- new net: D28.2 (A), MX28.2 (ROW)
- new net: D25.2 (A), MX25.2 (ROW)
- new net: D31.2 (A), MX31.2 (ROW)
- new net: D23.2 (A), MX23.2 (ROW)
- new net: D44.2 (A), MX44.2 (ROW)
- new net: D29.2 (A), MX29.2 (ROW)
- new net +5V: C1.1, C2.1, C3.1, C6.1, F1.2, R3.1, U1.14 (VCC), U1.2 (UVCC), U1.24 (AVCC), U1.34 (VCC), U1.44 (AVCC), U1.7 (VBUS)
- new net Col 0: MX1.1 (COL), MX2.1 (COL), MX3.1 (COL), MX4.1 (COL), U1.18 (PD0)
- new net Col 1: MX5.1 (COL), MX6.1 (COL), MX7.1 (COL), MX8.1 (COL), U1.19 (PD1)
- new net Col 10: MX39.1 (COL), MX40.1 (COL), MX41.1 (COL), MX42.1 (COL), U1.30 (PB6)
- new net Col 11: MX43.1 (COL), MX44.1 (COL), MX45.1 (COL), MX46.1 (COL), U1.31 (PC6)
- new net Col 2: MX10.1 (COL), MX11.1 (COL), MX12.1 (COL), MX9.1 (COL), U1.20 (PD2)
- new net Col 3: MX13.1 (COL), MX14.1 (COL), MX15.1 (COL), U1.21 (PD3)
- new net Col 4: MX16.1 (COL), MX17.1 (COL), MX18.1 (COL), MX19.1 (COL), U1.25 (PD4)
- new net Col 5: MX20.1 (COL), MX21.1 (COL), MX22.1 (COL), U1.22 (PD5)
- new net Col 6: MX23.1 (COL), MX24.1 (COL), MX25.1 (COL), MX26.1 (COL), U1.26 (PD6)
- new net Col 7: MX27.1 (COL), MX28.1 (COL), MX29.1 (COL), MX30.1 (COL), U1.27 (PD7)
- new net Col 8: MX31.1 (COL), MX32.1 (COL), MX33.1 (COL), MX34.1 (COL), U1.28 (PB4)
- new net Col 9: MX35.1 (COL), MX36.1 (COL), MX37.1 (COL), MX38.1 (COL), U1.29 (PB5)
- new net D+: J1.A6 (D+), J1.B6 (D+), R2.1
- new net D-: J1.A7 (D-), J1.B7 (D-), R1.1
- new net GND: C1.2, C2.2, C3.2, C4.1, C5.1, C6.2, C7.2, J1.A1 (GND), J1.A12 (GND), J1.B1 (GND), J1.B12 (GND), R4.2, R5.2, R6.2, SW1.1, SW2.C, U1.15 (GND), U1.23 (GND), U1.35 (GND), U1.43 (GND), U1.45 (GND), U1.5 (UGND), Y1.2, Y1.4
- new net Rot 0: SW2.A, U1.37 (PF6)
- new net Rot 1: SW2.B, U1.36 (PF7)
- new net Row 0: D1.1 (K), D13.1 (K), D16.1 (K), D20.1 (K), D23.1 (K), D27.1 (K), D31.1 (K), D35.1 (K), D39.1 (K), D43.1 (K), D5.1 (K), D9.1 (K), U1.8 (PB0)
- new net Row 1: D10.1 (K), D14.1 (K), D17.1 (K), D2.1 (K), D21.1 (K), D24.1 (K), D28.1 (K), D32.1 (K), D36.1 (K), D40.1 (K), D44.1 (K), D6.1 (K), U1.9 (PB1)
- new net Row 2: D11.1 (K), D15.1 (K), D18.1 (K), D22.1 (K), D25.1 (K), D29.1 (K), D3.1 (K), D33.1 (K), D37.1 (K), D41.1 (K), D45.1 (K), D7.1 (K), U1.11 (PB3)
- new net Row 3: D12.1 (K), D19.1 (K), D26.1 (K), D30.1 (K), D34.1 (K), D38.1 (K), D4.1 (K), D42.1 (K), D46.1 (K), D8.1 (K), U1.10 (PB2)
- new net VCC: F1.1, J1.A4 (VBUS), J1.A9 (VBUS), J1.B4 (VBUS), J1.B9 (VBUS)
